Commit message: test: make CAD golden robust to mesh-computed inertia
The golden URDFs were first generated in an incomplete environment (no
scipy / 3dxml loader), so build() emitted PLACEHOLDER inertials and the
snapshots baked those in. In a full environment build() computes real
inertia from the mesh, so the goldens failed.

Inertia is build()'s geometry maths -- not what the edit-overlay refactor
these goldens guard touches -- and its exact value varies with platform /
optional-dep availability. So normalize the <inertial> block away before
comparing (it has its own tests: test_autoinit, test_sw_inertia) and
re-baseline the snapshots to <inertial/>. The edit-driven structure
(names / types / limits / axis / mimic) is still asserted exactly.

Full suite now green with the complete env (skrobot/scipy/pycollada/
networkx/catkin_pkg): 177 passed, 7 skipped.

File: tests/golden/fingertip_base.urdf (robot description, URDF)
Before this commit: robot fingertip, 3 links, 2 joints
Links:
- link base_link: mass 0.1 -> None
- link fingertip_back_1: mass 0.1 -> None
- link screwlock_male_hard_jointbase_v4_1: mass 0.1 -> None

File: tests/golden/fingertip_edited.urdf (robot description, URDF)
Before this commit: robot fingertip, 3 links, 2 joints
Links:
- link base_link: mass 0.1 -> None
- link screwlock_male_hard_jointbase_v4_1: mass 0.1 -> None
- link tip: mass 0.1 -> None

File: tests/golden/fingertip_flip.urdf (robot description, URDF)
Before this commit: robot fingertip, 3 links, 2 joints
Links:
- link base_link: mass 0.1 -> None
- link fingertip_back_1: mass 0.1 -> None
- link screwlock_male_hard_jointbase_v4_1: mass 0.1 -> None

File: tests/golden/fingertip_rename_direct.urdf (robot description, URDF)
Before this commit: robot fingertip, 3 links, 2 joints
Links:
- link base_link: mass 0.1 -> None
- link screwlock_male_hard_jointbase_v4_1: mass 0.1 -> None
- link tip: mass 0.1 -> None
