Commit message: refactor: use scikit-robot math instead of hand-rolled transforms
Require scikit-robot>=0.3.27 and call matrix_relative / rpy2homogeneous /
matrix2xyzrpy directly at each call site; orthonormalize SolidWorks rotations
at the ArrayData entry point and share one strict URDF <origin> parser.

File: tests/golden/fingertip_base.urdf (robot description, URDF)
Before this commit: robot fingertip, 3 links, 2 joints
Joints:
- joint fingertip_front_2__fingertip_back_1: origin xyz=0.021039487 -0.0155 0.031 rpy=3.1415927 8.2450846e-17 8.2450846e-17 -> xyz=0.021039487 -0.0155 0.031 rpy=3.1415927 0 0
- joint fingertip_front_2__screwlock_male_hard_jointbase_v4_1: origin xyz=7.0484173e-18 -0.0155 0.038 rpy=1.5707963 -3.3306691e-16 -3.1415927 -> xyz=0 -0.0155 0.038 rpy=1.5707963 0 -3.1415927

File: tests/golden/fingertip_edited.urdf (robot description, URDF)
Before this commit: robot fingertip, 3 links, 2 joints
Joints:
- joint bend: origin xyz=0.021039487 -0.0155 0.031 rpy=3.1415927 8.2450846e-17 8.2450846e-17 -> xyz=0.021039487 -0.0155 0.031 rpy=3.1415927 0 0
- joint fingertip_front_2__screwlock_male_hard_jointbase_v4_1: origin xyz=4.2862638e-18 0.0015 0.035 rpy=3.1415927 8.2450846e-17 8.2450846e-17 -> xyz=0 0.0015 0.035 rpy=3.1415927 0 0

File: tests/golden/fingertip_flip.urdf (robot description, URDF)
Before this commit: robot fingertip, 3 links, 2 joints
Joints:
- joint fingertip_front_2__fingertip_back_1: origin xyz=0.021039487 -0.0155 0.031 rpy=3.1415927 8.2450846e-17 8.2450846e-17 -> xyz=0.021039487 -0.0155 0.031 rpy=3.1415927 0 0
- joint fingertip_front_2__screwlock_male_hard_jointbase_v4_1: origin xyz=7.0484173e-18 -0.0155 0.038 rpy=1.5707963 -3.3306691e-16 -3.1415927 -> xyz=0 -0.0155 0.038 rpy=1.5707963 0 -3.1415927

File: tests/golden/fingertip_rename_direct.urdf (robot description, URDF)
Before this commit: robot fingertip, 3 links, 2 joints
Joints:
- joint bend: origin xyz=0.021039487 -0.0155 0.031 rpy=3.1415927 8.2450846e-17 8.2450846e-17 -> xyz=0.021039487 -0.0155 0.031 rpy=3.1415927 0 0
- joint fingertip_front_2__screwlock_male_hard_jointbase_v4_1: origin xyz=7.0484173e-18 -0.0155 0.038 rpy=1.5707963 -3.3306691e-16 -3.1415927 -> xyz=0 -0.0155 0.038 rpy=1.5707963 0 -3.1415927

Commit message: refactor: one <origin> formatter and writer in exporter/geometry.py
Four modules each wrote URDF <origin> with their own float formatter
(%.10g, repr(round(v, 9)), %.8g twice), so the same coordinate printed
differently depending on which code path touched it last, and an editor
edit silently truncated an exported origin from 10 digits to 8.

fmt_urdf_num / fmt_urdf_vec / set_urdf_origin now live next to the
parser in exporter/geometry.py, and merge, urdf_writer, ros_export and
the editor all route through them.  %.10g is the precision: it is the
highest any call site used, so nothing is degraded, and origins are the
storage format for an editor edit -- they have to survive
write -> read -> write unchanged.

The formatter no longer rounds.  ros_export's old snap of |v| < 1e-9 to
"0" is dropped: matrix_to_xyz_rpy already snaps the BLAS-dependent SVD
noise it was covering, at 1e-12, and the other three writers printed
those values all along.

urdf_origin_matrix grows a strict= flag rather than keeping the editor's
second copy.  Strict (default) is for URDFs sw2robot wrote, where a
wrong-length xyz is an exporter bug; the editor passes strict=False
because it also opens hand-edited files.

Golden re-baselined on Linux: origins gain two significant digits (max
delta 4.6e-8 rad on a pi-valued rpy, 3.1e-10 m on xyz -- the digits the
old %.8g dropped), and <axis xyz="-0 -0 1"> prints as "0 0 1".

File: tests/golden/fingertip_base.urdf (robot description, URDF)
Before this commit: robot fingertip, 3 links, 2 joints
Joints:
- joint fingertip_front_2__fingertip_back_1: origin xyz=0.021039487 -0.0155 0.031 rpy=3.1415927 0 0 -> xyz=0.02103948669 -0.0155 0.031 rpy=3.141592654 0 0
- joint fingertip_front_2__screwlock_male_hard_jointbase_v4_1: axis -0 -0 1 -> 0 0 1; origin xyz=0 -0.0155 0.038 rpy=1.5707963 0 -3.1415927 -> xyz=0 -0.0155 0.038 rpy=1.570796327 0 -3.141592654

File: tests/golden/fingertip_edited.urdf (robot description, URDF)
Before this commit: robot fingertip, 3 links, 2 joints
Joints:
- joint bend: origin xyz=0.021039487 -0.0155 0.031 rpy=3.1415927 0 0 -> xyz=0.02103948669 -0.0155 0.031 rpy=3.141592654 0 0
- joint fingertip_front_2__screwlock_male_hard_jointbase_v4_1: axis 0 -1 -0 -> 0 -1 0; origin xyz=0 0.0015 0.035 rpy=3.1415927 0 0 -> xyz=0 0.0015 0.035 rpy=3.141592654 0 0

File: tests/golden/fingertip_flip.urdf (robot description, URDF)
Before this commit: robot fingertip, 3 links, 2 joints
Joints:
- joint fingertip_front_2__fingertip_back_1: origin xyz=0.021039487 -0.0155 0.031 rpy=3.1415927 0 0 -> xyz=0.02103948669 -0.0155 0.031 rpy=3.141592654 0 0
- joint fingertip_front_2__screwlock_male_hard_jointbase_v4_1: axis -0 -0 1 -> 0 0 1; origin xyz=0 -0.0155 0.038 rpy=1.5707963 0 -3.1415927 -> xyz=0 -0.0155 0.038 rpy=1.570796327 0 -3.141592654

File: tests/golden/fingertip_rename_direct.urdf (robot description, URDF)
Before this commit: robot fingertip, 3 links, 2 joints
Joints:
- joint bend: origin xyz=0.021039487 -0.0155 0.031 rpy=3.1415927 0 0 -> xyz=0.02103948669 -0.0155 0.031 rpy=3.141592654 0 0
- joint fingertip_front_2__screwlock_male_hard_jointbase_v4_1: axis -0 -0 1 -> 0 0 1; origin xyz=0 -0.0155 0.038 rpy=1.5707963 0 -3.1415927 -> xyz=0 -0.0155 0.038 rpy=1.570796327 0 -3.141592654
